File: pcb/74181_alu_tester.kicad_pcb (KiCad board)
At the start: 2 copper layers, 70 x 50 mm, 0 parts

Commit message: Add full 74181 tester PCB layout, Gerbers, and board preview.
Other:
- board text added: "74181 ALU tester 70x50mm Preview: pcb_render.png Fab: 74181_alu_tester_gerbers.zip Build: py -3 generate_board.py"
- board text removed: "74181 ALU tester 70x50mm Upload 74181_alu_tester_gerbers.zip to JLCPCB"
Changed lines of the file:
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@@
     (rev "1")
     (company "brightwaterfall")
-    (comment 1 "70x50mm 2-layer — Gerbers in gerbers/ and 74181_alu_tester_gerbers.zip")
-    (comment 2 "Regenerate: python generate_gerbers.py")
+    (comment 1 "70x50mm 2-layer — see pcb_render.png and 74181_alu_tester_gerbers.zip")
+    (comment 2 "Regenerate: py -3 generate_board.py")
   )
   (layers
@@
     (layer "Edge.Cuts")
   )
-  (gr_text "74181 ALU tester 70x50mm\nUpload 74181_alu_tester_gerbers.zip to JLCPCB"
+  (gr_text "74181 ALU tester 70x50mm\nPreview: pcb_render.png\nFab: 74181_alu_tester_gerbers.zip\nBuild: py -3 generate_board.py"
     (at 35 25)
     (layer "Cmts.User")
